File: SCRM6816.kicad_pcb (KiCad board)
At the start: 2 copper layers, 276.9 x 142.2 mm, 130 parts, among them J1 ramslot1, J10 perslot3ad, J11 perslot4ad, J12 perslot3c, J13 perslot4c, J14 peridcad, J15 peridcc, J16 pwrjack, J2 ramslot2, J3 ramslot3, J4 ramslot4, J6 perslot1ad, J7 perslot1c, J8 perslot2ad, J9 perslot2c, M2 MountingHole_3.2mm_M3_Pad, Q2 NPN, SW1 ressw, SW2 pwrsw, SW3 timersw, SW4 SW_DIP_x08, U1 68HC000P16, U10 28C256, U11 74HC157, U12 74HC157, U13 AS7C256C-15PCN, U14 74HC245, U15 AS7C256C-15PCN, U16 74HC245, U17 74HC541, U18 74HC541, U19 74HC541, U2 74HC04, U20 74HC541, U21 74HC688, U22 74HC573, U23 74HC541, U24 74HC08, U25 74HC273, U26 74HC14, U27 74HC541, U29 74HC32, U3 74HC688, U30 74HC139, U33 74HC541, U4 74HC688, U5 74HC4075, U56 74HC688, U57 74HC573, U58 74HC541, U6 74HC32, U7 74HC14, U8 74HC05, U9 28C256, X1 CXO_DIP8_16MHz

Commit message: routing: progress 1
Parts:
- moved U21 72.7 mm to (353.1, -185.4)
- moved B5 72.7 mm to (350.5, -193.0)
- moved C2 44.9 mm to (307.3, -195.6)
- moved U22 44.9 mm to (287.0, -185.4)
- moved R5 44.9 mm to (312.4, -195.6)
- moved B5 44.9 mm to (284.5, -193.0)
- moved B5 44.9 mm to (317.5, -193.0)
- moved U23 44.9 mm to (320.0, -185.4)
- moved U10 43.2 mm to (238.8, -177.8)
- moved U13 43.2 mm to (195.6, -154.9)
- moved B5 36.4 mm to (317.5, -162.6)
- moved B5 36.4 mm to (350.5, -162.6)
- moved U18 36.4 mm to (353.1, -154.9)
- moved B5 36.4 mm to (317.5, -177.8)
- moved B5 36.4 mm to (350.5, -177.8)
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Connections:
- J1 pad 13: /E_{8} -> /E_{0}
- J1 pad 15: /E_{10} -> /E_{2}
- J1 pad 16: /E_{9} -> /E_{1}
- J1 pad 17: /E_{12} -> /E_{4}
- J1 pad 18: /E_{11} -> /E_{3}
- J1 pad 19: /E_{14} -> /E_{6}
- J1 pad 20: /E_{13} -> /E_{5}
- J1 pad 21: /E_{0} -> /E_{8}
- J1 pad 22: /E_{15} -> /E_{7}
- J1 pad 24: /E_{1} -> /E_{9}
- J10 pad 13: /E_{8} -> /E_{0}
- J10 pad 15: /E_{10} -> /E_{2}
- J10 pad 16: /E_{9} -> /E_{1}
- J10 pad 17: /E_{12} -> /E_{4}
- J10 pad 18: /E_{11} -> /E_{3}
- J10 pad 19: /E_{14} -> /E_{6}
- J10 pad 20: /E_{13} -> /E_{5}
- J10 pad 21: /E_{0} -> /E_{8}
- J10 pad 22: /E_{15} -> /E_{7}
- J10 pad 23: /E_{2} -> /E_{10}
- J10 pad 24: /E_{1} -> /E_{9}
- J10 pad 26: /E_{3} -> /E_{11}
- J11 pad 13: /E_{8} -> /E_{0}
- J11 pad 15: /E_{10} -> /E_{2}
- J11 pad 16: /E_{9} -> /E_{1}
- J11 pad 17: /E_{12} -> /E_{4}
- J11 pad 18: /E_{11} -> /E_{3}
- J11 pad 19: /E_{14} -> /E_{6}
- J11 pad 20: /E_{13} -> /E_{5}
- J11 pad 21: /E_{0} -> /E_{8}
- J11 pad 22: /E_{15} -> /E_{7}
- J11 pad 23: /E_{2} -> /E_{10}
- J11 pad 24: /E_{1} -> /E_{9}
- J11 pad 26: /E_{3} -> /E_{11}
- J12 pad 4: /E_{5} -> /E_{13}
- J12 pad 6: /E_{6} -> /E_{14}
- J12 pad 8: /E_{7} -> /E_{15}
- J13 pad 4: /E_{5} -> /E_{13}
- J13 pad 6: /E_{6} -> /E_{14}
- J13 pad 8: /E_{7} -> /E_{15}
- J14 pad 25: /E_{3} -> /E_{11}
- J14 pad 27: /E_{1} -> /E_{9}
- J14 pad 28: /E_{2} -> /E_{10}
- J14 pad 29: /E_{15} -> /E_{7}
- J14 pad 30: /E_{0} -> /E_{8}
- J14 pad 31: /E_{13} -> /E_{5}
- J14 pad 32: /E_{14} -> /E_{6}
- J14 pad 33: /E_{11} -> /E_{3}
- J14 pad 34: /E_{12} -> /E_{4}
- J14 pad 35: /E_{9} -> /E_{1}
- J14 pad 36: /E_{10} -> /E_{2}
- J14 pad 38: /E_{8} -> /E_{0}
- J15 pad 23: /E_{7} -> /E_{15}
- J15 pad 25: /E_{6} -> /E_{14}
- J15 pad 27: /E_{5} -> /E_{13}
- J2 pad 13: /E_{8} -> /E_{0}
- J2 pad 15: /E_{10} -> /E_{2}
- J2 pad 16: /E_{9} -> /E_{1}
- J2 pad 17: /E_{12} -> /E_{4}
- J2 pad 18: /E_{11} -> /E_{3}
- J2 pad 19: /E_{14} -> /E_{6}
- J2 pad 20: /E_{13} -> /E_{5}
- J2 pad 21: /E_{0} -> /E_{8}
- J2 pad 22: /E_{15} -> /E_{7}
- J2 pad 24: /E_{1} -> /E_{9}
- J2 pad 44: /DRD -> /ram/~{BKE_{1}}
- J3 pad 13: /E_{8} -> /E_{0}
- J3 pad 15: /E_{10} -> /E_{2}
- J3 pad 16: /E_{9} -> /E_{1}
- J3 pad 17: /E_{12} -> /E_{4}
- J3 pad 18: /E_{11} -> /E_{3}
- J3 pad 19: /E_{14} -> /E_{6}
- J3 pad 20: /E_{13} -> /E_{5}
- J3 pad 21: /E_{0} -> /E_{8}
- J3 pad 22: /E_{15} -> /E_{7}
- J3 pad 24: /E_{1} -> /E_{9}
- J4 pad 13: /E_{8} -> /E_{0}
- J4 pad 15: /E_{10} -> /E_{2}
- J4 pad 16: /E_{9} -> /E_{1}
- J4 pad 17: /E_{12} -> /E_{4}
- J4 pad 18: /E_{11} -> /E_{3}
- J4 pad 19: /E_{14} -> /E_{6}
- J4 pad 20: /E_{13} -> /E_{5}
- J4 pad 21: /E_{0} -> /E_{8}
- J4 pad 22: /E_{15} -> /E_{7}
- J4 pad 24: /E_{1} -> /E_{9}
- J6 pad 13: /E_{8} -> /E_{0}
- J6 pad 15: /E_{10} -> /E_{2}
- J6 pad 16: /E_{9} -> /E_{1}
- J6 pad 17: /E_{12} -> /E_{4}
- J6 pad 18: /E_{11} -> /E_{3}
- J6 pad 19: /E_{14} -> /E_{6}
- J6 pad 20: /E_{13} -> /E_{5}
- J6 pad 21: /E_{0} -> /E_{8}
- J6 pad 22: /E_{15} -> /E_{7}
- J6 pad 23: /E_{2} -> /E_{10}
- J6 pad 24: /E_{1} -> /E_{9}
- J6 pad 26: /E_{3} -> /E_{11}
- J7 pad 4: /E_{5} -> /E_{13}
- J7 pad 6: /E_{6} -> /E_{14}
- J7 pad 8: /E_{7} -> /E_{15}
- J8 pad 13: /E_{8} -> /E_{0}
- J8 pad 15: /E_{10} -> /E_{2}
- J8 pad 16: /E_{9} -> /E_{1}
- J8 pad 17: /E_{12} -> /E_{4}
- J8 pad 18: /E_{11} -> /E_{3}
- J8 pad 19: /E_{14} -> /E_{6}
- J8 pad 20: /E_{13} -> /E_{5}
- J8 pad 21: /E_{0} -> /E_{8}
- J8 pad 22: /E_{15} -> /E_{7}
- J8 pad 23: /E_{2} -> /E_{10}
- J8 pad 24: /E_{1} -> /E_{9}
- J8 pad 26: /E_{3} -> /E_{11}
- J9 pad 4: /E_{5} -> /E_{13}
- J9 pad 6: /E_{6} -> /E_{14}
- J9 pad 8: /E_{7} -> /E_{15}
- U2 pad 10: /DIR.~{R} -> /statusreg/LD
- U2 pad 11: /DIR.~{W} -> Net-(U2-Pad11)
- U2 pad 8: /~{DRD} -> /atu/pidreg/LD
- U2 pad 9: /DRD -> Net-(U2-Pad9)
- U29 pad 1: /E_{6} -> /E_{14}
- U29 pad 5: /E_{5} -> /E_{13}
- U29 pad 9: /E_{7} -> /E_{15}
- U30 pad 2: /E_{2} -> /E_{11}
- U30 pad 3: /E_{3} -> /E_{10}
- U30 pad 5: /DRD -> /ram/~{BKE_{1}}
- U6 pad 11: Net-(U6-Pad11) -> Net-(U2-Pad11)
- U6 pad 8: Net-(U6-Pad8) -> Net-(U2-Pad9)
- U7 pad 5: Net-(U6-Pad8) -> /DRD
- U7 pad 6: /atu/pidreg/LD -> /~{DRD}
- U7 pad 8: /statusreg/LD -> /DIR.~{R}
- U7 pad 9: Net-(U6-Pad11) -> /DIR.~{W}
Routing:
- net /E_{4}: track 0.00 -> 338.1 mm, vias 0 -> 6
- net /E_{2}: track 75.4 -> 349.4 mm, vias 1 -> 6
- net /E_{6}: track 69.9 -> 337.3 mm, vias 0 -> 6
- net /atu/EA_{12}: track 0.00 -> 261.9 mm, vias 0 -> 4
- net /E_{3}: track 69.9 -> 325.7 mm, vias 0 -> 5
- net /E_{7}: track 69.9 -> 325.3 mm, vias 0 -> 5
- net /E_{5}: track 69.9 -> 324.9 mm, vias 0 -> 5
- net /D_{14}: track 122.8 -> 356.2 mm, vias 0 -> 7
- net /atu/EA_{14}: track 0.00 -> 233.2 mm, vias 0 -> 3
- net /D_{15}: track 135.6 -> 366.3 mm, vias 2 -> 7
- net /D_{12}: track 122.8 -> 348.6 mm, vias 0 -> 7
- net /D_{13}: track 135.6 -> 358.6 mm, vias 2 -> 8
- net /E_{0}: track 135.6 -> 351.7 mm, vias 2 -> 5
- net /D_{11}: track 135.6 -> 350.3 mm, vias 2 -> 6
- net /E_{1}: track 122.8 -> 336.6 mm, vias 0 -> 5
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
Commit message: connected ram slots to A & D bus
Parts:
- moved SW4 19.3 mm to (254.0, -63.5), turned to 90 degrees
Connections:
- SW4 pad 1: GND -> /statusreg/SI_{7}
- SW4 pad 10: /statusreg/SI_{6} -> GND
- SW4 pad 11: /statusreg/SI_{5} -> GND
- SW4 pad 12: /statusreg/SI_{4} -> GND
- SW4 pad 13: /statusreg/SI_{3} -> GND
- SW4 pad 14: /statusreg/SI_{2} -> GND
- SW4 pad 15: /statusreg/SI_{1} -> GND
- SW4 pad 16: /statusreg/SI_{0} -> GND
- SW4 pad 2: GND -> /statusreg/SI_{6}
- SW4 pad 3: GND -> /statusreg/SI_{5}
- SW4 pad 4: GND -> /statusreg/SI_{4}
- SW4 pad 5: GND -> /statusreg/SI_{3}
- SW4 pad 6: GND -> /statusreg/SI_{2}
- SW4 pad 7: GND -> /statusreg/SI_{1}
- SW4 pad 8: GND -> /statusreg/SI_{0}
- SW4 pad 9: /statusreg/SI_{7} -> GND
- U30 pad 1: /~{RIH} -> Net-(U30A-E)
- U30 pad 10: unconnected-(U30B-O2-Pad10) -> Net-(U30A-E)
- U30 pad 13: +5V -> /~{RIH}
- U30 pad 14: +5V -> /BE.~{M}
- U30 pad 15: +5V -> GND
Routing:
- net /D_{7}: track 196.2 -> 499.2 mm, vias 2 -> 8
- net /D_{6}: track 198.3 -> 493.8 mm, vias 2 -> 10
- net /D_{5}: track 210.9 -> 491.2 mm, vias 3 -> 7
- net /D_{4}: track 223.0 -> 475.8 mm, vias 1 -> 11
- net /D_{3}: track 229.9 -> 474.2 mm, vias 3 -> 8
- net /D_{2}: track 216.1 -> 458.5 mm, vias 3 -> 13
- net /D_{0}: track 193.2 -> 435.0 mm, vias 3 -> 12
- net /D_{1}: track 229.4 -> 457.7 mm, vias 5 -> 10
- net /A_{7}: track 262.4 -> 448.3 mm, vias 4 -> 17
- net /A_{5}: track 266.2 -> 450.9 mm, vias 3 -> 17
- net /A_{6}: track 270.9 -> 453.9 mm, vias 5 -> 13
- net /A_{3}: track 286.8 -> 447.6 mm, vias 4 -> 17
- net /A_{4}: track 294.5 -> 453.2 mm, vias 5 -> 14
- net /D_{10}: track 332.0 -> 490.2 mm, vias 5 -> 10
- net /D_{8}: track 328.7 -> 485.9 mm, vias 4 -> 9
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
Commit message: connected A16-23 to atu
Parts:
- added C12: 10uF, Capacitor_THT:CP_Radial_D5.0mm_P2.00mm, F.Cu at (367.0, -133.3)
- added C12: 10uF, Capacitor_THT:CP_Radial_D5.0mm_P2.00mm, F.Cu at (139.7, -121.9)
- added C12: 10uF, Capacitor_THT:CP_Radial_D5.0mm_P2.00mm, F.Cu at (403.9, -109.1)
- added C12: 10uF, Capacitor_THT:CP_Radial_D5.0mm_P2.00mm, F.Cu at (170.2, -121.9)
- moved M2 24.2 mm to (268.6, -215.3)
- moved C2 20.9 mm to (312.4, -215.9)
- moved R5 20.9 mm to (317.5, -215.9)
Routing:
- net /A_{19}: track 0.00 -> 307.1 mm, vias 0 -> 4
- net /A_{18}: track 0.00 -> 303.7 mm, vias 0 -> 4
- net /A_{17}: track 0.00 -> 299.9 mm, vias 0 -> 4
- net /A_{16}: track 0.00 -> 296.1 mm, vias 0 -> 4
- net /A_{23}: track 0.00 -> 280.2 mm, vias 0 -> 4
- net /A_{22}: track 0.00 -> 277.8 mm, vias 0 -> 4
- net /A_{21}: track 0.00 -> 275.6 mm, vias 0 -> 4
- net /A_{20}: track 0.00 -> 270.5 mm, vias 0 -> 4
- net /A_{12}: track 104.3 -> 343.3 mm, vias 2 -> 9
- net /A_{14}: track 102.4 -> 333.8 mm, vias 2 -> 13
- net /A_{15}: track 81.8 -> 281.9 mm, vias 2 -> 13
- net /A_{13}: track 86.9 -> 270.1 mm, vias 2 -> 12
- net /A_{10}: track 392.5 -> 438.1 mm, vias 4 -> 6
- net /A_{11}: track 395.0 -> 434.5 mm, vias 8 -> 12
- net /A_{9}: track 387.0 -> 424.6 mm, vias 7 -> 11
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