File: power&reset.kicad_sch (KiCad schematic)
At the start: 17 parts, among them J5 pwrjack, SW1 SW_Push, SW2 pwrsw, U55 L7805, U7 74HC14, U8 74HC05

Commit message: done the pcb layout + added the 1M ram bank project
Parts:
- removed C15: 10uF, Capacitor_THT:C_Radial_D5.0mm_H7.0mm_P2.00mm, symbol Device:C_Polarized
- removed D1: D_Filled, Diode_THT:D_DO-35_SOD27_P7.62mm_Horizontal, symbol Device:D_Filled
- removed J5: pwrjack, Connector_BarrelJack:BarrelJack_Horizontal, symbol Connector:Barrel_Jack_Switch
- removed U55: L7805, Package_TO_SOT_THT:TO-220-3_Horizontal_TabDown, symbol Regulator_Linear:L7805
- added C3: 100uF, Capacitor_THT:CP_Radial_D8.0mm_P3.50mm, symbol Device:C_Polarized
- added J16: pwrjack, Connector_BarrelJack:BarrelJack_Horizontal, symbol Connector:Barrel_Jack_Switch
- C12, C16: footprint Capacitor_THT:C_Radial_D5.0mm_H7.0mm_P2.00mm -> Capacitor_THT:CP_Radial_D5.0mm_P2.00mm
- C13, C14: footprint Capacitor_THT:C_Disc_P2.54mm -> Capacitor_THT:C_Disc_D3.0mm_W1.6mm_P2.54mm
- SW1: value SW_Push -> ressw; footprint Button_Switch_THT:SW_PUSH_6mm -> Connector_PinHeader_2.54mm:PinHeader_1x02_P2.54mm_Vertical
- U7, U8: footprint Package_DIP:DIP-14_W7.62mm_Socket -> Package_DIP:DIP-14_W7.62mm
Connections:
- net +9V is gone; now on net +5V: C12.1, C13.2, SW2.2 (B)
- net +5V: now also C3.1
- net GND: now also C3.2, J16.2, J16.3
- net at SW2.3 (C): now also J16.1
Other:
- moved on the sheet: C12, C13, C14, C16, D2, R1, R2, R22, R6, SW1, SW2, U7A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

Commit message: first commit: scheme ok [decoder]: 	- new spv. address space [mmu]: 	- removed pidreg 	- switched back to 8Kb mmu rams [ram/peripherals]: 	- added ground pins to connectors [misc]: 	- added DMA support 	- added clock halfer
Parts:
- removed C12, C16: 10uF, Capacitor_THT:CP_Radial_D5.0mm_P2.00mm, symbol Device:C_Polarized
- removed C13: 330nF, Capacitor_THT:C_Disc_D3.0mm_W1.6mm_P2.54mm, symbol Device:C
- removed C14: 100nF, Capacitor_THT:C_Disc_D3.0mm_W1.6mm_P2.54mm, symbol Device:C
- removed C3: 100uF, Capacitor_THT:CP_Radial_D8.0mm_P3.50mm, symbol Device:C_Polarized
- removed D2: LED_Filled, LED_THT:LED_D5.0mm, symbol Device:LED_Filled
- removed J16: pwrjack, Connector_BarrelJack:BarrelJack_Horizontal, symbol Connector:Barrel_Jack_Switch
- removed R1, R2: 4k7, Resistor_THT:R_Axial_DIN0207_L6.3mm_D2.5mm_P2.54mm_Vertical, symbol Device:R
- removed R22: 14k7, Resistor_THT:R_Axial_DIN0207_L6.3mm_D2.5mm_P2.54mm_Vertical, symbol Device:R
- removed R6: 1k, Resistor_THT:R_Axial_DIN0207_L6.3mm_D2.5mm_P2.54mm_Vertical, symbol Device:R
- removed SW1: ressw, Connector_PinHeader_2.54mm:PinHeader_1x02_P2.54mm_Vertical, symbol Switch:SW_Push
- removed SW2: pwrsw, Connector_PinHeader_2.54mm:PinHeader_1x03_P2.54mm_Vertical, symbol Switch:SW_SPDT
- removed U7: 74HC14, Package_DIP:DIP-14_W7.62mm, symbol 74xx:74HC14
- removed U8: 74HC05, Package_DIP:DIP-14_W7.62mm, symbol 74xx:74LS05
