File: atu_buffers.kicad_sch (KiCad schematic)
At the start: 6 parts, among them U14 74HC245, U16 74HC245, U17 74HC541, U18 74HC541, U19 74HC541, U20 74HC541

Commit message: done the pcb layout + added the 1M ram bank project
Parts:
- U14, U16, U17, U18, U19, U20: footprint Package_DIP:DIP-20_W7.62mm_Socket -> Package_DIP:DIP-20_W7.62mm
Changed lines of the file:
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@@
 			)
 		)
-		(property "Footprint" "Package_DIP:DIP-20_W7.62mm_Socket"
+		(property "Footprint" "Package_DIP:DIP-20_W7.62mm"
 			(at 241.3 63.5 0)
 			(effects
@@
 			)
 		)
-		(property "Footprint" "Package_DIP:DIP-20_W7.62mm_Socket"
+		(property "Footprint" "Package_DIP:DIP-20_W7.62mm"
 			(at 177.8 63.5 0)
 			(effects
@@
 			)
 		)
-		(property "Footprint" "Package_DIP:DIP-20_W7.62mm_Socket"
+		(property "Footprint" "Package_DIP:DIP-20_W7.62mm"
 			(at 50.8 127 0)
 			(effects
@@
 			)
 		)
-		(property "Footprint" "Package_DIP:DIP-20_W7.62mm_Socket"
+		(property "Footprint" "Package_DIP:DIP-20_W7.62mm"
 			(at 50.8 63.5 0)
 			(effects
@@
 			)
 		)
-		(property "Footprint" "Package_DIP:DIP-20_W7.62mm_Socket"
+		(property "Footprint" "Package_DIP:DIP-20_W7.62mm"
 			(at 114.3 127 0)
 			(effects
@@
 			)
 		)
-		(property "Footprint" "Package_DIP:DIP-20_W7.62mm_Socket"
+		(property "Footprint" "Package_DIP:DIP-20_W7.62mm"
 			(at 114.3 63.5 0)
 			(effects

Commit message: first commit: scheme ok [decoder]: 	- new spv. address space [mmu]: 	- removed pidreg 	- switched back to 8Kb mmu rams [ram/peripherals]: 	- added ground pins to connectors [misc]: 	- added DMA support 	- added clock halfer
Parts:
- added U23: 74HC04, symbol 74xx:74LS04
Connections:
- net PN_{0} is gone; now on net +5V: U20.6 (A4)
- net PN_{1} is gone; now on net +5V: U20.7 (A5)
- net PN_{2} is gone; now on net +5V: U20.8 (A6)
- net +5V: now also U18.6 (A4), U18.7 (A5), U18.8 (A6)
- net A_{13}: no longer U18.6 (A4)
- net A_{14}: no longer U18.7 (A5)
- net A_{15}: no longer U18.8 (A6)
- net EA_{12}: no longer names the net of U20.14 (Y4)
- net EA_{12}: no longer U18.14 (Y4)
- net EA_{13}: no longer names the net of U20.13 (Y5)
- net EA_{13}: no longer U18.13 (Y5)
- net EA_{14}: no longer names the net of U20.12 (Y6)
- net EA_{14}: no longer U18.12 (Y6)
- net MOD.~{R} renamed S/~{R}
- net S/~{R}: now also U23.10
- net MOD.~{S} renamed R/~{S}
- net R/~{S}: now also U23.11
- no-connect marks 2 -> 8
Other:
- moved on the sheet: U14, U16, U17, U18, U19, U20

Commit message: assigned footprints
Parts:
- U23: footprint (none) -> Package_DIP:DIP-14_W7.62mm
Changed lines of the file:
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@@
 			)
 		)
-		(property "Footprint" ""
+		(property "Footprint" "Package_DIP:DIP-14_W7.62mm"
 			(at 50.8 38.1 0)
 			(effects
