File: SF68.kicad_pcb (KiCad board)
At the start: 4 copper layers, 271.8 x 147.3 mm, 130 parts, among them J1 perslot4a, J10 perslot4b, J11 perslot3b, J12 perslot2b, J13 perslot1b, J14 pwrjack, J15 perslot5b, J16 stprobe, J2 perslot3a, J3 perslot2a, J4 perslot1a, J5 ramslot1, J6 ramslot2, J7 ramslot3, J8 perslot5a, J9 ramslot4, M1 MountingHole_3.2mm_M3_DIN965_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, M2 MountingHole_3.2mm_M3_DIN965_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, M3 MountingHole_3.2mm_M3_DIN965_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, M4 MountingHole_3.2mm_M3_DIN965_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, M5 MountingHole_3.2mm_M3_DIN965_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, M6 MountingHole_3.2mm_M3_DIN965_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, Q1 Q_NPN_CBE, SW1 pwrsw, SW2 ressw, SW3 timersw, U1 74HC541, U10 AS7C164A, U11 68HC000P10, U12 74HC688, U13 74HC157, U14 74HC74, U15 74HC688, U16 74HC139, U17 74HC04, U18 74HC688, U19 74HC32, U2 74HC541, U20 74HC541, U21 74HC32, U22 74HC05, U23 74HC32, U24 74HC273, U25 74HC08, U26 74HC541, U27 74HC14, U28 74HC08, U29 74HC541, U3 74HC245, U30 74HC14, U4 28C256, U5 28C256, U6 74HC541, U7 74HC541, U8 74HC245, U9 AS7C164A, X1 CXO_DIP8

Commit message: 1.0.0 commit
Parts:
- C1: value 22pF -> 220pF
- JP2: value romdrd -> romrd
- R11: value 20k -> 2k
Changed lines of the file:
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@@
 			(crossoutdnponfab yes)
 			(subtractmaskfromsilk no)
-			(outputformat 1)
+			(outputformat 5)
 			(mirror no)
 			(drillshape 0)
 			(scaleselection 1)
-			(outputdirectory "")
+			(outputdirectory "svg/")
 		)
 	)
@@
 			)
 		)
-		(property "Value" "22pF"
+		(property "Value" "220pF"
 			(at 1.27 2.05 0)
 			(layer "F.Fab")
@@
 			)
 		)
-		(property "Value" "romdrd"
+		(property "Value" "romrd"
 			(at 0 4.92 90)
 			(layer "F.Fab")
@@
 			)
 		)
-		(property "Value" "20k"
+		(property "Value" "2k"
 			(at 1.27 2.37 0)
 			(layer "F.Fab")
