File: rom.kicad_sch (KiCad schematic)
At the start: 3 parts, among them U10 28C256, U6 74HC32, U9 28C256

Commit message: 1.0.0 commit
Parts:
- added C1: 220pF, Capacitor_THT:C_Disc_D3.0mm_W1.6mm_P2.54mm, symbol Device:C
- added JP2: romrd, Connector_PinHeader_2.54mm:PinHeader_1x02_P2.54mm_Vertical, symbol Jumper:Jumper_2_Open
- added R11: 2k, Resistor_THT:R_Axial_DIN0207_L6.3mm_D2.5mm_P2.54mm_Vertical, symbol Device:R
- added U22: 74HC05, Package_DIP:DIP-14_W7.62mm, symbol 74xx:74LS05
- added U27: 74HC14, Package_DIP:DIP-14_W7.62mm, symbol 74xx:74HC14
- renumbered U6 to U19, U9 to U4, U10 to U5
Connections:
- net +5V: now also U19.10, U19.9; no longer U19.12, U19.13
- net BE.~{EE}: now also U27.5
- net GND: now also R11.2
- new net: JP2.1 (A), U22.6
- new net: C1.2, R11.1, U22.5
- new net: C1.1, U27.6
- new net DRD: JP2.2 (B)
