File: vga/vga.kicad_sch (KiCad schematic)
At the start: 52 parts, among them J13 perslotb, J4 perslota, U1 74HC161, U10 74HC541, U11 74HC541, U12 74HC541, U13 74HC541, U14 74HC541, U15 74HC541, U16 74HC541, U17 74HC541, U18 74HC541, U19 74HC574, U2 74HC161, U20 74HC541, U21 74HC541, U22 AS6C4008-55PCN, U23 74HC541, U24 74HC541, U25 74HC245, U26 74HC245, U27 74HC574, U28 74HC541, U29 74HC541, U3 74HC161, U30 74HC541, U31 74HC541, U32 74HC541, U33 74HC574, U34 74HC574, U35 74HC574, U36 74HC245, U37 74HC245, U38 AS6C4008-55PCN, U39 AS6C4008-55PCN, U4 74HC161, U40 74HC574, U41 74HC574, U42 74HC541, U43 74HC541, U44 74HC161, U45 74HC73, U48 74HC04, U5 74HC161, U55 74HC08, U56 74HC11, U57 74HC21, U6 AS6C4008-55PCN, U7 74HC574, U8 74HC574, U9 74HC574, Y1 CXO_DIP8_25.175MHz

Commit message: lcd2x16 ready
Parts:
- removed J13: perslotb, Connector_PCBEdge:55308432, symbol Connector_Generic:Conn_02x15_Odd_Even
- removed J4: perslota, Connector_TE-Connectivity:55308437, symbol Connector_Generic:Conn_02x30_Odd_Even
- removed U1, U2, U3, U4, U44, U5: 74HC161, symbol 74xx:74LS161
- removed U10, U11, U12, U13, U14, U15, U16, U17, U18, U20, U21, U23, U24, U28, U29, U30, U31, U32, U42, U43: 74HC541, symbol 74xx:74AHC541
- removed U19, U27, U33, U34, U35, U40, U41, U7, U8, U9: 74HC574, symbol 74xx:74HCT574
- removed U22, U38, U39, U6: AS6C4008-55PCN, Package_DIP:DIP-32_W15.24mm, symbol Memory_RAM:AS6C4008-55PCN
- removed U25, U26, U36, U37: 74HC245, symbol 74xx:74HC245
- removed U45: 74HC73, symbol 74xx:74LS73
- removed U48: 74HC04, symbol 74xx:74HC04
- removed U55: 74HC08, symbol 74xx:74LS08
- removed U56: 74HC11, symbol 74xx:74LS11
- removed U57: 74HC21, symbol 74xx:74LS21
- removed Y1: CXO_DIP8_25.175MHz, Oscillator:Oscillator_DIP-8, symbol Oscillator:CXO_DIP8
Connections:
- no-connect marks 55 -> 0
Other:
- added sheet banks (banks.kicad_sch)
- added sheet banks_addr_muxes (banks_addr_muxes.kicad_sch)
- added sheet banks_data_demuxes (banks_data_demuxes.kicad_sch)
- added sheet bus_connector (bus_connector.kicad_sch)
- added sheet bus_mapper (bus_mapper.kicad_sch)
- added sheet color_muxes (color_muxes.kicad_sch)
- added sheet control_reg (control_reg.kicad_sch)
- added sheet counters (counters.kicad_sch)
- added sheet vga_interface (vga_interface.kicad_sch)
- note added: "pixel mode pipeline: (2 cycles wide) (consider the following happening 'in parallel') - fetched pixels are latched; - rams start fetching the next 2 pixels; - the latched pixels are shown multiplexed by col-counter's bit 0. characters mode pipeline: (8 cycles wide) - fetched bitmap byte (by rom) is latched; - rams start fetching the character word; - rom starts fetching the bitmap once the rams a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"
- note removed: "0010 0111 1110 0010 1000 1110 0010 1110 1110 0011 0001 1111 t0 = A123 t1 = A56 Bj = t0 * t1 * A49 t2 = t0 * B Sj = t2 * !t1 Sk = t2 * t1 Bk = t2 * A048"
- note removed: "horizontal, unit = pixel, '->' = clocked: 0x27e: active video -> blank, front porch 0x28e: front porch -> sync 0x2ee: sync -> back porch 0x31e: backporch -> active video, reset counter"
- note removed: "vertical, unit = scanline: 0x1E0: active video -> blank, front porch 0x1EA: front porch -> sync 0x1EC: sync -> back porch 0x20D: back porch -> active video, reset counter"
