File: vga/bus_connector.kicad_sch (KiCad schematic)
At the start: 2 parts, among them J1 perslota, J3 perslotb

Commit message: [vga]	added logos + fixed jtag version
Parts:
- renumbered J1 to J2, J3 to J5
Changed lines of the file:
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@@
 		(on_board yes)
 		(dnp no)
-		(property "Reference" "J3"
+		(property "Reference" "J5"
 			(at 139.7 182.88 0)
 			(effects
@@
 			(project "vga_cpld"
 				(path "/eac05228-afcc-4a64-b0a2-d2674f34b0cf/0cc2963d-7dd2-477c-a8d8-221ca822480e"
-					(reference "J3")
+					(reference "J5")
 					(unit 1)
 				)
@@
 		(on_board yes)
 		(dnp no)
-		(property "Reference" "J1"
+		(property "Reference" "J2"
 			(at 139.7 132.08 0)
 			(effects
@@
 			(project "vga_cpld"
 				(path "/eac05228-afcc-4a64-b0a2-d2674f34b0cf/0cc2963d-7dd2-477c-a8d8-221ca822480e"
-					(reference "J1")
-					(unit 1)
-				)
+					(reference "J2")
+					(unit 1)
+				)
