File: vga/vga_cpld.kicad_pcb (KiCad board)
At the start: 2 copper layers, 223.5 x 147.3 mm, 121 parts, among them J1 perslota, J2 vgasupply, J3 perslotb, J4 DE15_Socket_HighDensity, M1 MountingHole_3.2mm_M3_DIN965_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, M2 MountingHole_3.2mm_M3_DIN965_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, M3 MountingHole_3.2mm_M3_DIN965_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, M4 MountingHole_3.2mm_M3_DIN965_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, Q1 Q_PNP_CBE, Q2 Q_NPN_CBE, U1 74AHC541, U10 74AHC541, U11 AS6C4008-55PCN, U12 AS6C4008-55PCN, U13 74AHC541, U14 74AHC541, U15 74HC157, U16 74HC157, U17 ATF1508AS-xJx84, U18 74AHC541, U19 74AHC541, U2 74AHC541, U20 ATF1502AS-xJx44, U21 74AHC541, U22 74AHC541, U23 AT28C16, U24 74HC541, U25 74AHC541, U26 74AHC541, U27 LM6171xxN, U28 LM6171xxN, U29 LM6171xxN, U3 AS6C4008-55PCN, U30 LM6172, U31 74AHC541, U32 74AHC541, U4 AS6C4008-55PCN, U5 74HC245, U6 74HC245, U7 74AHC541, U8 74HC245, U9 74HC245, Y1 CXO_DIP8_25.175MHz

Commit message: [vga]:	added +12V & GND labels on 12V supply connector
Other:
- board text added: "+12V"
- board text added: "-12V"
- board text added: "GND"
Changed lines of the file:
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@@
 		(layer "Edge.Cuts")
+	)
+	(gr_text "GND"
+		(at 266.7 -139.7 0)
+		(layer "F.SilkS")
+		(effects
+			(font
+				(size 1.27 1.143)
+				(thickness 0.142875)
+			)
+			(justify right)
+		)
+	)
+	(gr_text "+12V"
+		(at 266.7 -142.24 0)
+		(layer "F.SilkS")
+		(effects
+			(font
+				(size 1.27 1.143)
+				(thickness 0.142875)
+			)
+			(justify right)
+		)
 	)
 	(gr_text "VGA Extension\n640x480@60Hz"
@@
 		)
 	)
+	(gr_text "-12V"
+		(at 266.7 -137.16 0)
+		(layer "F.SilkS")
+		(effects
+			(font
+				(size 1.27 1.143)
+				(thickness 0.142875)
+			)
+			(justify right)
+		)
+	)

Commit message: [vga]	added logos + fixed jtag version
Parts:
- added B19: 100n, Capacitor_THT:C_Disc_D3.0mm_W1.6mm_P2.54mm, F.Cu at (149.9, -200.7)
- added B23: 100n, Capacitor_THT:C_Disc_D3.0mm_W1.6mm_P2.54mm, F.Cu at (91.4, -185.4)
- added C6: 100u, Capacitor_THT:CP_Radial_D8.0mm_P3.50mm, F.Cu at (115.6, -180.3)
- added G***: LOGO, LOGO, F.Cu at (256.5, -217.2)
- moved C4 14.8 mm to (127.0, -172.7), turned to 0 degrees
Routing:
- net /~{VS}: track 222.3 -> 220.8 mm
- net /CM: track 71.9 -> 70.4 mm
Other:
- board text added: "640x480@60Hz"
- board text added: "Copyright © 2026 Pietro Senesi, Italy"
- board text added: "SF68"
- board text added: "VGA Extension"
- board text removed: "VGA Extension 640x480@60Hz"
