File: vga/vga_cpld_jtag.kicad_pcb (KiCad board)
At the start: 2 copper layers, 223.5 x 147.3 mm, 123 parts, among them J1 perslota, J2 vgasupply, J3 perslotb, J4 DE15_Socket_HighDensity, J5 jtag, M1 MountingHole_3.2mm_M3_DIN965_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, M2 MountingHole_3.2mm_M3_DIN965_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, M3 MountingHole_3.2mm_M3_DIN965_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, M4 MountingHole_3.2mm_M3_DIN965_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, Q1 Q_PNP_CBE, Q2 Q_NPN_CBE, U1 74AHC541, U10 74AHC541, U11 AS6C4008-55PCN, U12 AS6C4008-55PCN, U13 74AHC541, U14 74AHC541, U15 74HC157, U16 74HC157, U17 ATF1508AS-xJx84, U18 74AHC541, U19 74AHC541, U2 74AHC541, U20 ATF1502AS-xJx44, U21 74AHC541, U22 74AHC541, U23 AT28C16, U24 74HC541, U25 74AHC541, U26 74AHC541, U27 LM6171xxN, U28 LM6171xxN, U29 LM6171xxN, U3 AS6C4008-55PCN, U30 LM6172, U31 74AHC541, U32 74AHC541, U4 AS6C4008-55PCN, U5 74HC245, U6 74HC245, U7 74AHC541, U8 74HC245, U9 74HC245, Y1 CXO_DIP8_25.175MHz

Commit message: [vga]	added logos + fixed jtag version
Parts:
- added C5: 10u, Capacitor_THT:CP_Radial_D5.0mm_P2.00mm, F.Cu at (127.0, -172.7)
- added G***: LOGO, LOGO, F.Cu at (256.5, -217.2)
- added J3: oe1_12v_bypass, Connector_PinHeader_2.54mm:PinHeader_2x01_P2.54mm_Vertical, F.Cu at (96.5, -154.9)
- added R9: 1k, Resistor_THT:R_Axial_DIN0207_L6.3mm_D2.5mm_P7.62mm_Horizontal, F.Cu at (99.1, -154.9)
- added RN1: 10k, Resistor_THT:R_Array_SIP6, F.Cu at (121.9, -175.3)
- moved C6 8.16 mm to (135.2, -172.7)
- moved Y1 2.54 mm to (129.5, -180.3)
- renumbered B19 to B17, B17 to B18, B18 to B19, B19 to B20, B20 to B21, B21 to B22, B22 to B23, B23 to B24, B24 to B25, B25 to B26, B26 to B27, B27 to B28, B28 to B29, B29 to B30, B30 to B31, B31 to B32, B32 to B33, B33 to B34, B34 to B35, B35 to B36, B36 to B37, C7 to C4, C4 to C6, C8 to C7, C5 to C8, C6 to C9, J5 to J1, J1 to J2, J2 to J4, J3 to J5, J4 to J6, Q2 to Q1, Q1 to Q2, R8 to R10, R9 to R11, R10 to R12, R11 to R13, R12 to R14, R13 to R15, R14 to R16, R15 to R17, R16 to R18, R17 to R19, R34 to R20, R18 to R21, R19 to R22, R20 to R23, R21 to R24, R22 to R25, R23 to R26, R24 to R27, R25 to R28, R26 to R29, R27 to R30, R28 to R31, R29 to R32, R30 to R33, R31 to R34, R32 to R35, R33 to R5, R5 to R6, R6 to R7, R7 to R8
Connections:
- net Net-(U17-I/O/TDO) renamed /08to02
- U17 pad 84: unconnected-(U17-I/OE1-Pad84) -> OE1_+12V
- U20 pad 44: unconnected-(U20-I/OE1-Pad44) -> OE1_+12V
Routing:
- net OE1_+12V: track 0.00 -> 122.8 mm, vias 0 -> 5
- net /08to02: track 112.5 -> 127.7 mm, vias 5 -> 6
- net /JTAG.TDI: track 70.2 -> 80.7 mm
- net /JTAG.TDO: track 26.0 -> 34.7 mm
- net /JTAG.TMS: track 131.4 -> 140.1 mm
- net /JTAG.TCK: track 109.7 -> 118.4 mm
- net Net-(J3-Pin_1): track 0.00 -> 2.54 mm
- net /CLK: track 25.4 -> 22.9 mm
- net +5V: track 135.4 -> 137.7 mm
- net GND: track 278.9 -> 280.2 mm
- net /DIR.~{W}: track 206.2 -> 206.9 mm
Other:
- board text added: "640x480@60Hz"
- board text added: "Copyright © 2026 Pietro Senesi, Italy"
- board text added: "SF68"
- board text added: "VGA Extension"
- board text removed: "VGA Extension 640x480@60Hz"
