File: vga/vga_cpld_jtag.kicad_sch (KiCad schematic)
At the start: 10 parts, among them J5 jtag, U15 74HC157, U16 74HC157, U17 ATF1508AS-xJx84, U20 ATF1502AS-xJx44, U23 AT28C16, U24 74HC541, Y1 CXO_DIP8_25.175MHz

Commit message: [vga]	added logos + fixed jtag version
Parts:
- added J3: oe1_12v_bypass, Connector_PinHeader_2.54mm:PinHeader_2x01_P2.54mm_Vertical, symbol Connector_Generic:Conn_02x01
- added R9: 1k, Resistor_THT:R_Axial_DIN0207_L6.3mm_D2.5mm_P7.62mm_Horizontal, symbol Device:R
- added RN1: 10k, Resistor_THT:R_Array_SIP6, symbol Device:R_Network05
- renumbered C5 to C8, J5 to J1, R14 to R16
Connections:
- net +5V: now also RN1.1 (common)
- net GND: now also J3.2 (Pin_2)
- net JTAG.TCK: now also RN1.6 (R5)
- net JTAG.TDI: now also RN1.2 (R1)
- net JTAG.TDO: now also RN1.5 (R4)
- net JTAG.TMS: now also RN1.4 (R3)
- net 08to02: now reaches U17.71 (I/O/TDO), U20.7 (I/O/TDI)
- net 08to02: now also RN1.3 (R2)
- net OE1_+12V: now reaches U17.84 (I/OE1)
- net OE1_+12V: now also U20.44 (I/OE1), R9.2
- new net: J3.1 (Pin_1), R9.1
- no-connect marks 17 -> 15
Other:
- moved on the sheet: J1
