File: vga/vga_interface.kicad_sch (KiCad schematic)
At the start: 43 parts, among them J2 vgasupply, J4 DE15_Socket_HighDensity, Q1 Q_PNP_CBE, Q2 Q_NPN_CBE, U27 LM6171xxN, U28 LM6171xxN, U29 LM6171xxN, U30 LM6172

Commit message: [vga]	added logos + fixed jtag version
Parts:
- renumbered C7 to C4, C8 to C7, J2 to J4, J4 to J6, Q2 to Q1, Q1 to Q2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
