File: ata/ata.kicad_sch (KiCad schematic)
At the start: 3 parts, among them J1 ata, J2 perslota, J3 perslotb

Commit message: [ata] started, but i think its destined to not go on.
Parts:
- added U1: 74HC04, symbol 74xx:74HC04
- added U2: 74HC541, symbol 74xx:74LS541
- added U3, U4: 74HC32, symbol 74xx:74LS32
- J1: footprint (none) -> Connector_IDC:IDC-Header_2x20_P2.54mm_Horizontal
Connections:
- net ADR_{0} is gone; now on net A_{1}: J1.35 (Pin_35)
- net ADR_{1} is gone; now on net A_{2}: J1.33 (Pin_33)
- net ADR_{2} is gone; now on net A_{3}: J1.36 (Pin_36)
- net RDY is gone; now on net DRD: J1.27 (Pin_27)
- net ~{R} is gone; now on net ~{RD}: J1.25 (Pin_25)
- net ~{W} is gone; now on net ~{WR}: J1.23 (Pin_23)
- net +5V: now also U2.20 (VCC), U2.3 (A1), U2.5 (A3), U2.8 (A6)
- net A_{4}: now also U1.3, U4.1
- net A_{5}: now also U1.1
- net A_{6}: now also U3.2
- net A_{7}: now also U3.1
- net GND: now also U2.10 (GND), U2.2 (A0), U2.4 (A2), U2.6 (A4), U2.7 (A5), U2.9 (A7)
- net IBSY: now also U2.19 (G2)
- net IRQ: now also U1.5
- net IRQ_{0}: now also U2.18 (Y0)
- net IRQ_{1}: now also U2.17 (Y1)
- net IRQ_{2}: now also U2.16 (Y2)
- net IRQ_{3}: now also U2.15 (Y3)
- net IRQ_{4}: now also U2.14 (Y4)
- net IRQ_{5}: now also U2.13 (Y5)
- net IRQ_{6}: now also U2.12 (Y6)
- net IRQ_{7}: now also U2.11 (Y7)
- net ~{CS1FX}: now also U4.3
- net ~{CS3FX}: now also U4.6
- net ~{RD}: now also U4.11; no longer J2.8 (Pin_8)
- net ~{US}: now also U3.13
- net ~{WR}: now also U4.8; no longer J2.7 (Pin_7)
- net DRD: now reaches J2.2 (Pin_2)
- net A_{10}: no longer names the net of J2.47 (Pin_47)
- net A_{11}: no longer names the net of J2.48 (Pin_48)
- net A_{12}: no longer names the net of J2.45 (Pin_45)
- net A_{13}: no longer names the net of J2.43 (Pin_43)
- net A_{14}: no longer names the net of J2.44 (Pin_44)
- net A_{15}: no longer names the net of J2.41 (Pin_41)
- net A_{16}: no longer names the net of J2.42 (Pin_42)
- net A_{17}: no longer names the net of J2.39 (Pin_39)
- net A_{18}: no longer names the net of J2.37 (Pin_37)
- net A_{19}: no longer names the net of J2.38 (Pin_38)
- net A_{20}: no longer names the net of J2.35 (Pin_35)
- net A_{21}: no longer names the net of J2.36 (Pin_36)
- net A_{22}: no longer names the net of J2.33 (Pin_33)
- net A_{23}: no longer names the net of J2.32 (Pin_32)
- net A_{8}: no longer names the net of J2.49 (Pin_49)
- net A_{9}: no longer names the net of J2.50 (Pin_50)
- net ~{IOEN} renamed ~{IOS}
- net ~{IOS}: now also U3.5
- new net: U1.6, U2.1 (G1)
- new net: U1.2, U3.4
- new net: U3.10, U3.6
- new net: U3.3, U3.9
- new net: U3.11, U4.10, U4.12
- new net: U1.4, U4.5
- new net ~{CS}: U3.12, U3.8, U4.2, U4.4
- new net ~{HRD}: J2.8 (Pin_8), U4.13
- new net ~{HWR}: J2.7 (Pin_7), U4.9
- no-connect marks 21 -> 36
Other:
- note added: "irq 0ah, lvl. 2/3"
- note added: "module decoder( _IOS, HADR, _CS, _US, _HWR, _HRD, _CS1FX, _CS3FX, _WR, _RD ); input _IOS; input [7:4] HADR; output _CS; input _US; input _HWR, _HRD; output _CS1FX, _CS3FX; output _WR, _RD; /* 0xCx to 0xDx */ assign _CS = !(HADR[7:5] == 0b110) | _IOS; assign _CS1FX = _CS | HADR[4]; assign _CS3FX = _CS | !HADR[4]; assign _WR = _CS | _US | _HWR; assign _RD = _CS | _US | _HRD; endmodule"
- moved on the sheet: J1
