File: vga/fctlines/vga_interface.kicad_sch (KiCad schematic)
At the start: 24 parts, among them J3 vga_connector, U23 CY74FCT244, U28 CY74FCT244

Commit message: [vga/fctlines] corrected errors on schematic. Schematic & PCB are NO longer matching.
Parts:
- R21, R9: value 294 -> 100
- R4: value 226 -> 100
Other:
- note added: "Last resistors should be 294 for 3bit dacs & 226 for 2bit, in order to correctly output 700mV. They've been lowered in order to prevent some signal smoothing."
Changed lines of the file:
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@@
 	(generator_version "9.0")
 	(paper "A4")
+	(text "Last resistors should be 294\nfor 3bit dacs & 226 for 2bit,\nin order to correctly output 700mV.\nThey've been lowered in order to\nprevent some signal smoothing."
+		(exclude_from_sim no)
+		(at 63.5 50.8 0)
+		(effects
+			(font
+				(size 1.27 1.27)
+			)
+			(justify left top)
+		)
+	)
 	(junction
 		(at 81.28 88.9)
@@
 			)
 		)
-		(property "Value" "226"
+		(property "Value" "100"
 			(at 189.23 76.2 90)
 			(effects
@@
 			)
 		)
-		(property "Value" "294"
+		(property "Value" "100"
 			(at 87.63 76.2 90)
 			(effects
@@
 			)
 		)
-		(property "Value" "294"
+		(property "Value" "100"
 			(at 138.43 76.2 90)
 			(effects
