File: vga/fctlines/vga_interface.kicad_sch (KiCad schematic)
At the start: 24 parts, among them J3 vga_connector, U23 CY74FCT244, U28 CY74FCT244

Commit message: [vga/fctlines] commit after a LONG time, i don't remember what i changed
Changed lines of the file:
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@@
 	(text "Last resistors should be 294\nfor 3bit dacs & 226 for 2bit,\nin order to correctly output 700mV.\nThey've been lowered in order to\nprevent some signal smoothing."
 		(exclude_from_sim no)
-		(at 63.5 50.8 0)
+		(at 63.5 114.3 0)
 		(effects
 			(font
@@
 	(wire
 		(pts
-			(xy 38.1 33.02) (xy 40.64 33.02)
+			(xy 63.5 58.42) (xy 66.04 58.42)
 		)
 		(stroke
@@
 	(wire
 		(pts
-			(xy 38.1 30.48) (xy 40.64 30.48)
+			(xy 63.5 55.88) (xy 66.04 55.88)
 		)
 		(stroke
@@
 	(bus
 		(pts
-			(xy 38.1 25.4) (xy 40.64 25.4)
+			(xy 63.5 50.8) (xy 66.04 50.8)
 		)
 		(stroke
@@
 	)
 	(label "~{HS}"
-		(at 40.64 30.48 0)
+		(at 66.04 55.88 0)
 		(effects
 			(font
@@
 	)
 	(label "~{VS}"
-		(at 40.64 33.02 0)
+		(at 66.04 58.42 0)
 		(effects
 			(font
@@
 	(hierarchical_label "~{HS}"
 		(shape input)
-		(at 38.1 30.48 180)
+		(at 63.5 55.88 180)
 		(effects
 			(font
@@
 	(hierarchical_label "RGB_{[0..7]}"
 		(shape input)
-		(at 38.1 25.4 180)
+		(at 63.5 50.8 180)
 		(effects
 			(font
@@
 	(hierarchical_label "~{VS}"
 		(shape input)
-		(at 38.1 33.02 180)
-		(effects
-			(font
+		(at 63.5 58.42 180)
+		(effects
+			(font
