File: vga/fctlines/bus_connector.kicad_sch (KiCad schematic)
At the start: 2 parts, among them J1 perslota, J2 perslotb

Commit message: [vga/fctlines] commit after a LONG time, i don't remember what i changed
Parts:
- removed J1: perslota, Connector_IDC:IDC-Header_2x30_P2.54mm_Horizontal, symbol Connector_Generic:Conn_02x30_Odd_Even
- removed J2: perslotb, Connector_IDC:IDC-Header_2x15_P2.54mm_Horizontal, symbol Connector_Generic:Conn_02x15_Odd_Even
Connections:
- no-connect marks 12 -> 0
