File: vga/fctlines/datacross.kicad_sch (KiCad schematic)
At the start: 9 parts, among them U1 74AHC541, U10 74AHC541, U2 74AHC541, U31 74HC32, U5 74HC245, U6 74HC245, U7 74AHC541, U8 74HC245, U9 74HC245

Commit message: [vga/fctlines] commit after a LONG time, i don't remember what i changed
Changed lines of the file:
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@@
 	(wire
 		(pts
-			(xy 38.1 33.02) (xy 40.64 33.02)
+			(xy 76.2 33.02) (xy 78.74 33.02)
 		)
 		(stroke
@@
 	(bus
 		(pts
-			(xy 48.26 27.94) (xy 50.8 27.94)
+			(xy 86.36 27.94) (xy 88.9 27.94)
 		)
 		(stroke
@@
 	(wire
 		(pts
-			(xy 38.1 38.1) (xy 40.64 38.1)
-		)
-		(stroke
-			(width 0)
-			(type default)
-		)
-	)
-	(wire
-		(pts
-			(xy 38.1 35.56) (xy 40.64 35.56)
+			(xy 76.2 38.1) (xy 78.74 38.1)
+		)
+		(stroke
+			(width 0)
+			(type default)
+		)
+	)
+	(wire
+		(pts
+			(xy 76.2 35.56) (xy 78.74 35.56)
 		)
 		(stroke
@@
 	(bus
 		(pts
-			(xy 38.1 27.94) (xy 40.64 27.94)
+			(xy 76.2 27.94) (xy 78.74 27.94)
 		)
 		(stroke
@@
 	(bus
 		(pts
-			(xy 38.1 25.4) (xy 40.64 25.4)
+			(xy 76.2 25.4) (xy 78.74 25.4)
 		)
 		(stroke
@@
 	(bus
 		(pts
-			(xy 48.26 25.4) (xy 50.8 25.4)
+			(xy 86.36 25.4) (xy 88.9 25.4)
 		)
 		(stroke
@@
 	)
 	(label "SEL"
-		(at 40.64 33.02 0)
+		(at 78.74 33.02 0)
 		(effects
 			(font
@@
 	)
 	(label "~{SEL}"
-		(at 40.64 35.56 0)
+		(at 78.74 35.56 0)
 		(effects
 			(font
@@
 	)
 	(label "DIR_{Y}"
-		(at 40.64 38.1 0)
+		(at 78.74 38.1 0)
 		(effects
 			(font
@@
 	(hierarchical_label "B_{[0..15]}"
 		(shape bidirectional)
-		(at 38.1 27.94 180)
+		(at 76.2 27.94 180)
 		(effects
 			(font
@@
 	(hierarchical_label "A_{[0..15]}"
 		(shape bidirectional)
-		(at 38.1 25.4 180)
+		(at 76.2 25.4 180)
 		(effects
 			(font
@@
 	(hierarchical_label "~{SEL}"
 		(shape input)
-		(at 38.1 35.56 180)
+		(at 76.2 35.56 180)
 		(effects
 			(font
@@
 	(hierarchical_label "Y_{[0..15]}"
 		(shape bidirectional)
-		(at 50.8 27.94 0)
+		(at 88.9 27.94 0)
 		(effects
 			(font
@@
 	(hierarchical_label "X_{[0..15]}"
 		(shape output)
-		(at 50.8 25.4 0)
+		(at 88.9 25.4 0)
 		(effects
 			(font
@@
 	(hierarchical_label "DIR_{Y}"
 		(shape input)
-		(at 38.1 38.1 180)
+		(at 76.2 38.1 180)
 		(effects
 			(font
@@
 	(hierarchical_label "SEL"
 		(shape input)
-		(at 38.1 33.02 180)
-		(effects
-			(font
+		(at 76.2 33.02 180)
+		(effects
+			(font
