File: vga/fctlines/vga_cpld_fctlines.kicad_sch (KiCad schematic)
At the start: 9 parts, among them U15 74HC157, U16 74HC157, U17 ATF1508AS-xJx84, U20 ATF1502AS-xJx44, U24 AT28C16, U25 74HC541, Y1 CXO_DIP8_25.175MHz

Commit message: [vga/fctlines] commit after a LONG time, i don't remember what i changed
Parts:
- added J1: perslota, Connector_IDC:IDC-Header_2x30_P2.54mm_Horizontal, symbol Connector_Generic:Conn_02x30_Odd_Even
- added J2: perslotb, Connector_IDC:IDC-Header_2x15_P2.54mm_Horizontal, symbol Connector_Generic:Conn_02x15_Odd_Even
Connections:
- net +5V: now also J1.1 (Pin_1), J1.31 (Pin_31), J1.59 (Pin_59), J2.1 (Pin_1), J2.29 (Pin_29)
- net AC.~{P}: now also J2.26 (Pin_26)
- net A_{19}: now also J1.38 (Pin_38)
- net A_{1}: now also J1.60 (Pin_60)
- net A_{20}: now also J1.35 (Pin_35)
- net A_{21}: now also J1.36 (Pin_36)
- net A_{22}: now also J1.33 (Pin_33)
- net A_{23}: now also J1.32 (Pin_32)
- net A_{2}: now also J1.57 (Pin_57)
- net A_{3}: now also J1.55 (Pin_55)
- net A_{4}: now also J1.56 (Pin_56)
- net A_{5}: now also J1.53 (Pin_53)
- net A_{6}: now also J1.54 (Pin_54)
- net A_{7}: now also J1.51 (Pin_51)
- net BE.~{IO}: now also J1.12 (Pin_12)
- net BE.~{M}: now also J1.9 (Pin_9)
- net DIR.~{R}: now also J1.8 (Pin_8)
- net DIR.~{W}: now also J1.7 (Pin_7)
- net DS.~{L}: now also J1.6 (Pin_6)
- net DS.~{U}: now also J1.5 (Pin_5)
- net D_{10}: now also J1.17 (Pin_17)
- net D_{11}: now also J1.18 (Pin_18)
- net D_{8}: now also J1.19 (Pin_19)
- net D_{9}: now also J1.20 (Pin_20)
- net GND: now also J1.10 (Pin_10), J1.16 (Pin_16), J1.22 (Pin_22), J1.28 (Pin_28), J1.34 (Pin_34), J1.4 (Pin_4), J1.40 (Pin_40), J1.46 (Pin_46), J1.52 (Pin_52), J1.58 (Pin_58), J2.10 (Pin_10), J2.16 (Pin_16), J2.21 (Pin_21), J2.22 (Pin_22), J2.28 (Pin_28), J2.4 (Pin_4)
- net IBSY: now also J2.2 (Pin_2)
- net IRQ_{0}: now also J2.11 (Pin_11)
- net IRQ_{1}: now also J2.12 (Pin_12)
- net IRQ_{2}: now also J2.9 (Pin_9)
- net IRQ_{3}: now also J2.7 (Pin_7)
- net IRQ_{4}: now also J2.8 (Pin_8)
- net IRQ_{5}: now also J2.5 (Pin_5)
- net IRQ_{6}: now also J2.6 (Pin_6)
- net IRQ_{7}: now also J2.3 (Pin_3)
- net ~{RES}: now also J2.13 (Pin_13)
- net ~{RIH}: now also J1.3 (Pin_3)
- new net A_{10}: J1.47 (Pin_47)
- new net A_{11}: J1.48 (Pin_48)
- new net A_{12}: J1.45 (Pin_45)
- new net A_{13}: J1.43 (Pin_43)
- new net A_{14}: J1.44 (Pin_44)
- new net A_{15}: J1.41 (Pin_41)
- new net A_{16}: J1.42 (Pin_42)
- new net A_{17}: J1.39 (Pin_39)
- new net A_{18}: J1.37 (Pin_37)
- new net A_{8}: J1.49 (Pin_49)
- new net A_{9}: J1.50 (Pin_50)
- new net D_{0}: J1.29 (Pin_29)
- new net D_{12}: J1.15 (Pin_15)
- new net D_{13}: J1.13 (Pin_13)
- new net D_{14}: J1.14 (Pin_14)
- new net D_{15}: J1.11 (Pin_11)
- new net D_{1}: J1.30 (Pin_30)
- new net D_{2}: J1.27 (Pin_27)
- new net D_{3}: J1.25 (Pin_25)
- new net D_{4}: J1.26 (Pin_26)
- new net D_{5}: J1.23 (Pin_23)
- new net D_{6}: J1.24 (Pin_24)
- new net D_{7}: J1.21 (Pin_21)
- no-connect marks 22 -> 34
Other:
- removed sheet bus_connector
- moved on the sheet: U15, U16, U20
