File: vga/fctlines/vram.kicad_sch (KiCad schematic)
At the start: 4 parts, among them U11 AS6C4008-55PCN, U12 AS6C4008-55PCN, U3 AS6C4008-55PCN, U4 AS6C4008-55PCN

Commit message: [vga/fctlines] commit after a LONG time, i don't remember what i changed
Changed lines of the file:
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@@
 	(bus
 		(pts
-			(xy 48.26 25.4) (xy 50.8 25.4)
+			(xy 73.66 25.4) (xy 76.2 25.4)
 		)
 		(stroke
@@
 	(bus
 		(pts
-			(xy 38.1 33.02) (xy 40.64 33.02)
+			(xy 63.5 33.02) (xy 66.04 33.02)
 		)
 		(stroke
@@
 	(bus
 		(pts
-			(xy 38.1 27.94) (xy 40.64 27.94)
+			(xy 63.5 27.94) (xy 66.04 27.94)
 		)
 		(stroke
@@
 	(bus
 		(pts
-			(xy 38.1 25.4) (xy 40.64 25.4)
+			(xy 63.5 25.4) (xy 66.04 25.4)
 		)
 		(stroke
@@
 	(bus
 		(pts
-			(xy 38.1 35.56) (xy 40.64 35.56)
+			(xy 63.5 35.56) (xy 66.04 35.56)
 		)
 		(stroke
@@
 	(bus
 		(pts
-			(xy 48.26 33.02) (xy 50.8 33.02)
+			(xy 73.66 33.02) (xy 76.2 33.02)
 		)
 		(stroke
@@
 	(hierarchical_label "VB_{1}A_{[0..17]}"
 		(shape input)
-		(at 38.1 33.02 180)
+		(at 63.5 33.02 180)
 		(effects
 			(font
@@
 	(hierarchical_label "VB_{0}D_{[0..15]}"
 		(shape bidirectional)
-		(at 50.8 25.4 0)
+		(at 76.2 25.4 0)
 		(effects
 			(font
@@
 	(hierarchical_label "VB_{1}D_{[0..15]}"
 		(shape bidirectional)
-		(at 50.8 33.02 0)
+		(at 76.2 33.02 0)
 		(effects
 			(font
@@
 	(hierarchical_label "VB_{1}C{~{E_{L}},~{E_{U}},~{R},~{W}}"
 		(shape input)
-		(at 38.1 35.56 180)
+		(at 63.5 35.56 180)
 		(effects
 			(font
@@
 	(hierarchical_label "VB_{0}A_{[0..17]}"
 		(shape input)
-		(at 38.1 25.4 180)
+		(at 63.5 25.4 180)
 		(effects
 			(font
@@
 	(hierarchical_label "VB_{0}C{~{E_{L}},~{E_{U}},~{R},~{W}}"
 		(shape input)
-		(at 38.1 27.94 180)
-		(effects
-			(font
+		(at 63.5 27.94 180)
+		(effects
+			(font
